File: Univerzalni_testovaci_platforma_nejen_pro_IoT_v1/_autosave-untitled.kicad_sch (KiCad schematic)
At the start: 6 parts, among them J1 Conn_01x22_Female ESP S3 J1, J2 Conn_01x22_Female ESP S3 J3, J3 Conn_01x19_Female ESP DEV_KIT, J4 Conn_01x19_Female ESP DEV_KIT, U1 ESP32-S3

Commit message: průběžný commit
Connections:
- net ESP S3 J1 pin10: now also U1.10 (GPIO17-TX1)
- net ESP S3 J1 pin11: now also U1.11 (GPIO18-RX1)
- net ESP S3 J1 pin12: now also U1.12 (GPIO8)
- net ESP S3 J1 pin13: now also U1.13 (GPIO3!!!D)
- net ESP S3 J1 pin14: now also U1.14 (GPIO46!!!D)
- net ESP S3 J1 pin15: now also U1.15 (GPIO9)
- net ESP S3 J1 pin16: now also U1.16 (GPIO10)
- net ESP S3 J1 pin17: now also U1.17 (GPIO11)
- net ESP S3 J1 pin18: now also U1.18 (GPIO12)
- net ESP S3 J1 pin19: now also U1.19 (GPIO13)
- net ESP S3 J1 pin20: now also U1.20 (GPIO14)
- net ESP S3 J1 pin4: now also U1.26 (GPIO1), U1.4 (GPIO4)
- net ESP S3 J1 pin5: now also U1.27 (GPIO2), U1.5 (GPIO5)
- net ESP S3 J1 pin6: now also U1.6 (GPIO6)
- net ESP S3 J1 pin7: now also U1.7 (GPIO7)
- net ESP S3 J1 pin8: now also U1.8 (GPIO15-RTS0)
- net ESP S3 J1 pin9: now also U1.9 (GPIO16-CTS0)
- net ESP S3 J3 pin10: now also U1.32 (GPIO38)
- net ESP S3 J3 pin11: now also U1.33 (GPIO37)
- net ESP S3 J3 pin12: now also U1.34 (GPIO36)
- net ESP S3 J3 pin13: now also U1.35 (GPIO35)
- net ESP S3 J3 pin14: now also U1.36 (GPIO0!!!U)
- net ESP S3 J3 pin15: now also U1.37 (GPIO45!!!D)
- net ESP S3 J3 pin16: now also U1.38 (GPIO48)
- net ESP S3 J3 pin17: now also U1.39 (GPIO47)
- net ESP S3 J3 pin18: now also U1.40 (GPIO21)
- net ESP S3 J3 pin19: now also U1.41 (GPIO20-D+)
- net ESP S3 J3 pin2: now also U1.24 (GPIO43-TX0)
- net ESP S3 J3 pin20: now also U1.42 (GPIO19-D-)
- net ESP S3 J3 pin3: now also U1.25 (GPIO44-RX0)
- net ESP S3 J3 pin6: now also U1.28 (GPIO42)
- net ESP S3 J3 pin7: now also U1.29 (GPIO41)
- net ESP S3 J3 pin8: now also U1.30 (GPIO40)
- net ESP S3 J3 pin9: now also U1.31 (GPIO39)
Changed lines of the file:
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@@
     (effects (font (size 1.27 1.27)) (justify left bottom))
   )
+  (hierarchical_label "ESP S3 J1 pin4" (shape input) (at 84.455 111.76 0)
+    (effects (font (size 1.27 1.27)) (justify left))
+  )
   (hierarchical_label "ESP DEV_KIT J2 pin10" (shape input) (at 184.785 45.085 180)
     (effects (font (size 1.27 1.27)) (justify right))
   )
+  (hierarchical_label "ESP S3 J1 pin17" (shape input) (at 84.455 137.16 0)
+    (effects (font (size 1.27 1.27)) (justify left))
+  )
   (hierarchical_label "ESP DEV_KIT J2 pin18" (shape input) (at 184.785 65.405 180)
     (effects (font (size 1.27 1.27)) (justify right))
@@
     (effects (font (size 1.27 1.27)) (justify left))
   )
+  (hierarchical_label "ESP S3 J3 pin10" (shape input) (at 84.455 162.56 0)
+    (effects (font (size 1.27 1.27)) (justify left))
+  )
+  (hierarchical_label "ESP S3 J1 pin13" (shape input) (at 53.975 127 180)
+    (effects (font (size 1.27 1.27)) (justify right))
+  )
   (hierarchical_label "ESP S3 J1 pin7" (shape input) (at 74.93 51.435 180)
     (effects (font (size 1.27 1.27)) (justify right))
   )
+  (hierarchical_label "ESP S3 J1 pin16" (shape input) (at 84.455 134.62 0)
+    (effects (font (size 1.27 1.27)) (justify left))
+  )
   (hierarchical_label "ESP DEV_KIT J3 pin4" (shape input) (at 123.825 27.305 0)
     (effects (font (size 1.27 1.27)) (justify left))
   )
+  (hierarchical_label "ESP S3 J3 pin14" (shape input) (at 53.975 124.46 180)
+    (effects (font (size 1.27 1.27)) (justify right))
+  )
   (hierarchical_label "ESP DEV_KIT J3 pin17" (shape input) (at 123.825 60.325 0)
     (effects (font (size 1.27 1.27)) (justify left))
@@
     (effects (font (size 1.27 1.27)) (justify left))
   )
+  (hierarchical_label "ESP S3 J3 pin7" (shape input) (at 84.455 170.18 0)
+    (effects (font (size 1.27 1.27)) (justify left))
+  )
   (hierarchical_label "ESP S3 J1 pin12" (shape input) (at 74.93 64.135 180)
     (effects (font (size 1.27 1.27)) (justify right))
@@
     (effects (font (size 1.27 1.27)) (justify left))
   )
+  (hierarchical_label "ESP S3 J3 pin16" (shape input) (at 84.455 180.34 0)
+    (effects (font (size 1.27 1.27)) (justify left))
+  )
+  (hierarchical_label "ESP S3 J1 pin9" (shape input) (at 53.975 149.86 180)
+    (effects (font (size 1.27 1.27)) (justify right))
+  )
   (hierarchical_label "ESP S3 J3 pin17" (shape input) (at 30.48 78.105 0)
     (effects (font (size 1.27 1.27)) (justify left))
   )
+  (hierarchical_label "ESP S3 J1 pin4" (shape input) (at 84.455 119.38 0)
+    (effects (font (size 1.27 1.27)) (justify left))
+  )
   (hierarchical_label "ESP DEV_KIT J3 pin16" (shape input) (at 123.825 57.785 0)
     (effects (font (size 1.27 1.27)) (justify left))
@@
     (effects (font (size 1.27 1.27)) (justify right))
   )
+  (hierarchical_label "ESP S3 J3 pin17" (shape input) (at 84.455 177.8 0)
+    (effects (font (size 1.27 1.27)) (justify left))
+  )
   (hierarchical_label "ESP S3 J1 pin17" (shape input) (at 74.93 76.835 180)
     (effects (font (size 1.27 1.27)) (justify right))
   )
+  (hierarchical_label "ESP S3 J3 pin18" (shape input) (at 84.455 149.86 0)
+    (effects (font (size 1.27 1.27)) (justify left))
+  )
   (hierarchical_label "ESP S3 J1 pin5" (shape input) (at 74.93 46.355 180)
     (effects (font (size 1.27 1.27)) (justify right))
@@
     (effects (font (size 1.27 1.27)) (justify left))
   )
+  (hierarchical_label "ESP S3 J1 pin6" (shape input) (at 84.455 124.46 0)
+    (effects (font (size 1.27 1.27)) (justify left))
+  )
   (hierarchical_label "ESP DEV_KIT J2 pin9" (shape input) (at 184.785 42.545 180)
     (effects (font (size 1.27 1.27)) (justify right))
   )
+  (hierarchical_label "ESP S3 J3 pin13" (shape input) (at 84.455 154.94 0)
+    (effects (font (size 1.27 1.27)) (justify left))
+  )
   (hierarchical_label "ESP DEV_KIT J2 pin13" (shape input) (at 184.785 52.705 180)
     (effects (font (size 1.27 1.27)) (justify right))
@@
     (effects (font (size 1.27 1.27)) (justify left))
   )
+  (hierarchical_label "ESP S3 J3 pin3" (shape input) (at 53.975 144.78 180)
+    (effects (font (size 1.27 1.27)) (justify right))
+  )
+  (hierarchical_label "ESP S3 J1 pin19" (shape input) (at 84.455 142.24 0)
+    (effects (font (size 1.27 1.27)) (justify left))
+  )
   (hierarchical_label "ESP DEV_KIT J2 pin17" (shape input) (at 184.785 62.865 180)
     (effects (font (size 1.27 1.27)) (justify right))
@@
     (effects (font (size 1.27 1.27)) (justify right))
   )
+  (hierarchical_label "ESP S3 J1 pin7" (shape input) (at 84.455 127 0)
+    (effects (font (size 1.27 1.27)) (justify left))
+  )
   (hierarchical_label "ESP S3 J3 pin8" (shape input) (at 30.48 55.245 0)
     (effects (font (size 1.27 1.27)) (justify left))
@@
     (effects (font (size 1.27 1.27)) (justify left))
   )
+  (hierarchical_label "ESP S3 J1 pin18" (shape input) (at 84.455 139.7 0)
+    (effects (font (size 1.27 1.27)) (justify left))
+  )
   (hierarchical_label "ESP DEV_KIT J2 pin6" (shape input) (at 184.785 34.925 180)
     (effects (font (size 1.27 1.27)) (justify right))
@@
     (effects (font (size 1.27 1.27)) (justify left))
   )
+  (hierarchical_label "ESP S3 J3 pin15" (shape input) (at 53.975 132.08 180)
+    (effects (font (size 1.27 1.27)) (justify right))
+  )
+  (hierarchical_label "ESP S3 J3 pin2" (shape input) (at 53.975 142.24 180)
+    (effects (font (size 1.27 1.27)) (justify right))
+  )
+  (hierarchical_label "ESP S3 J3 pin12" (shape input) (at 84.455 157.48 0)
+    (effects (font (size 1.27 1.27)) (justify left))
+  )
+  (hierarchical_label "ESP S3 J1 pin20" (shape input) (at 84.455 144.78 0)
+    (effects (font (size 1.27 1.27)) (justify left))
+  )
   (hierarchical_label "ESP DEV_KIT J3 pin10" (shape input) (at 123.825 42.545 0)
     (effects (font (size 1.27 1.27)) (justify left))
@@
     (effects (font (size 1.27 1.27)) (justify right))
   )
+  (hierarchical_label "ESP S3 J1 pin10" (shape input) (at 53.975 152.4 180)
+    (effects (font (size 1.27 1.27)) (justify right))
+  )
+  (hierarchical_label "ESP S3 J3 pin8" (shape input) (at 84.455 167.64 0)
+    (effects (font (size 1.27 1.27)) (justify left))
+  )
+  (hierarchical_label "ESP S3 J1 pin8" (shape input) (at 53.975 147.32 180)
+    (effects (font (size 1.27 1.27)) (justify right))
+  )
   (hierarchical_label "ESP S3 J1 pin16" (shape input) (at 74.93 74.295 180)
     (effects (font (size 1.27 1.27)) (justify right))
@@
     (effects (font (size 1.27 1.27)) (justify left))
   )
+  (hierarchical_label "ESP S3 J1 pin14" (shape input) (at 53.975 129.54 180)
+    (effects (font (size 1.27 1.27)) (justify right))
+  )
   (hierarchical_label "ESP S3 J1 pin10" (shape input) (at 74.93 59.055 180)
     (effects (font (size 1.27 1.27)) (justify right))
@@
     (effects (font (size 1.27 1.27)) (justify right))
   )
+  (hierarchical_label "ESP S3 J1 pin5" (shape input) (at 84.455 121.92 0)
+    (effects (font (size 1.27 1.27)) (justify left))
+  )
   (hierarchical_label "ESP DEV_KIT J3 pin5" (shape input) (at 123.825 29.845 0)
     (effects (font (size 1.27 1.27)) (justify left))
@@
     (effects (font (size 1.27 1.27)) (justify left))
   )
+  (hierarchical_label "ESP S3 J1 pin11" (shape input) (at 53.975 154.94 180)
+    (effects (font (size 1.27 1.27)) (justify right))
+  )
+  (hierarchical_label "ESP S3 J3 pin6" (shape input) (at 84.455 172.72 0)
+    (effects (font (size 1.27 1.27)) (justify left))
+  )
+  (hierarchical_label "ESP S3 J3 pin9" (shape input) (at 84.455 165.1 0)
+    (effects (font (size 1.27 1.27)) (justify left))
+  )
   (hierarchical_label "ESP S3 J3 pin13" (shape input) (at 30.48 67.945 0)
     (effects (font (size 1.27 1.27)) (justify left))
@@
     (effects (font (size 1.27 1.27)) (justify left))
   )
+  (hierarchical_label "ESP S3 J3 pin20" (shape input) (at 53.975 137.16 180)
+    (effects (font (size 1.27 1.27)) (justify right))
+  )
+  (hierarchical_label "ESP S3 J3 pin19" (shape input) (at 53.975 139.7 180)
+    (effects (font (size 1.27 1.27)) (justify right))
+  )
   (hierarchical_label "ESP DEV_KIT J2 pin8" (shape input) (at 184.785 40.005 180)
     (effects (font (size 1.27 1.27)) (justify right))
@@
     (effects (font (size 1.27 1.27)) (justify left))
   )
+  (hierarchical_label "ESP S3 J1 pin15" (shape input) (at 84.455 132.08 0)
+    (effects (font (size 1.27 1.27)) (justify left))
+  )
+  (hierarchical_label "ESP S3 J3 pin11" (shape input) (at 84.455 160.02 0)
+    (effects (font (size 1.27 1.27)) (justify left))
+  )
   (hierarchical_label "ESP S3 J1 pin13" (shape input) (at 74.93 66.675 180)
     (effects (font (size 1.27 1.27)) (justify right))
@@
     (effects (font (size 1.27 1.27)) (justify left))
   )
+  (hierarchical_label "ESP S3 J1 pin12" (shape input) (at 84.455 129.54 0)
+    (effects (font (size 1.27 1.27)) (justify left))
+  )
   (hierarchical_label "ESP S3 J1 pin14" (shape input) (at 74.93 69.215 180)
     (effects (font (size 1.27 1.27)) (justify right))
@@
     (effects (font (size 1.27 1.27)) (justify left))
   )
+  (hierarchical_label "ESP S3 J1 pin5" (shape input) (at 84.455 114.3 0)
+    (effects (font (size 1.27 1.27)) (justify left))
+  )
