File: Univerzalni_testovaci_platforma_nejen_pro_IoT_v1/Univerzalni_testovaci_platforma_nejen_pro_IoT_v1.kicad_sch (KiCad schematic)
At the start: 110 parts, among them J3 Conn_01x19_Female ESP DEV_KIT, J4 Conn_01x19_Female ESP DEV_KIT, J5 Conn_02x03_Counter_Clockwise, J6 USB_C_Receptacle, J7 Conn_02x10_Odd_Even, J8 Conn_02x10_Odd_Even, SW1 SW_Push_Dual, U1 STM32F103ZETx, U2 AMS1117CS-3.3, Y1 12Mhz

Commit message: průběžný commit
Parts:
- removed J3, J4: Conn_01x19_Female ESP DEV_KIT, Connector_PinSocket_2.54mm:PinSocket_1x19_P2.54mm_Vertical, symbol Connector:Conn_01x19_Female
Other:
- moved on the sheet: J7

Commit message: schema hotovo
Parts:
- removed J7, J8: Conn_02x10_Odd_Even, Connector_PinHeader_2.54mm:PinHeader_2x10_P2.54mm_Vertical, symbol Connector_Generic:Conn_02x10_Odd_Even
- removed SW1: SW_Push_Dual, Button_Switch_SMD:SW_SPST_TL3342, symbol Switch:SW_Push_Dual
- removed U2: AMS1117CS-3.3, Package_TO_SOT_SMD:TO-252-2, symbol Regulator_Linear:AMS1117CS-3.3
- added H1, H2, H3, H4: MountingHole, MountingHole:MountingHole_3.2mm_M3, symbol Mechanical:MountingHole
- added J1, J10, J11, J12, J2, J3, J4, J7, J8, J9: Conn_01x10_Male, Connector_PinHeader_2.54mm:PinHeader_1x10_P2.54mm_Vertical, symbol Connector:Conn_01x10_Male
- added SW1: SW_MEC_5E, symbol Switch:SW_MEC_5E
- added U2: AMS1117-3.3, Package_TO_SOT_SMD:TO-252-2, symbol Regulator_Linear:AMS1117-3.3
- added U3: ESP32-DEVKITC-32D, robotarna:MODULE_ESP32-DEVKITC-32D, symbol robotarna_sym:ESP32-DEVKITC-32D
- added U4: ESP32-S3, robotarna1:ESP32-devkit_v1, symbol Robotarna_KiCad_Library:ESP32-S3
- J6: LCSC (none) -> C165948
Connections:
- net +3V3: now also R79.1, J11.1 (Pin_1), J11.10 (Pin_10), J11.2 (Pin_2), J11.3 (Pin_3), J11.4 (Pin_4), J11.5 (Pin_5), J11.6 (Pin_6), J11.7 (Pin_7), J11.8 (Pin_8), J11.9 (Pin_9), J12.1 (Pin_1), J12.10 (Pin_10), J12.2 (Pin_2), J12.3 (Pin_3), J12.4 (Pin_4), J12.5 (Pin_5), J12.6 (Pin_6), J12.7 (Pin_7), J12.8 (Pin_8), J12.9 (Pin_9), U2.2 (VO)
- net +5V: now also U2.3 (VI); no longer R79.1
- net GND: now also J3.1 (Pin_1), J3.10 (Pin_10), J3.2 (Pin_2), J3.3 (Pin_3), J3.4 (Pin_4), J3.5 (Pin_5), J3.6 (Pin_6), J3.7 (Pin_7), J3.8 (Pin_8), J3.9 (Pin_9), J4.1 (Pin_1), J4.10 (Pin_10), J4.2 (Pin_2), J4.3 (Pin_3), J4.4 (Pin_4), J4.5 (Pin_5), J4.6 (Pin_6), J4.7 (Pin_7), J4.8 (Pin_8), J4.9 (Pin_9), J8.1 (Pin_1), J8.10 (Pin_10), J8.2 (Pin_2), J8.3 (Pin_3), J8.4 (Pin_4), J8.5 (Pin_5), J8.6 (Pin_6), J8.7 (Pin_7), J8.8 (Pin_8), J8.9 (Pin_9), J9.1 (Pin_1), J9.10 (Pin_10), J9.2 (Pin_2), J9.3 (Pin_3), J9.4 (Pin_4), J9.5 (Pin_5), J9.6 (Pin_6), J9.7 (Pin_7), J9.8 (Pin_8), J9.9 (Pin_9), SW1.1, SW1.2, U2.1 (GND), U3.J2-14 (GND1), U3.J3-1 (GND3), U3.J3-7 (GND2), U4.22 (GND), U4.23 (GND), U4.43 (GND), U4.44 (GND)
- net PA10: now also J2.1 (Pin_1)
- net PA13: now also J2.2 (Pin_2)
- net PA14: now also J2.3 (Pin_3)
- net PA15: now also J2.4 (Pin_4)
- net PB0: now also J2.5 (Pin_5)
- net PB1: now also J2.6 (Pin_6)
- net PC4: now also J2.7 (Pin_7)
- net PC5: now also J2.8 (Pin_8)
- net PC6: now also J2.9 (Pin_9)
- net PC7: now also J2.10 (Pin_10)
- net PC8: now also J7.1 (Pin_1)
- net PD10: now also J7.3 (Pin_3)
- net PD11: now also J7.4 (Pin_4)
- net PD12: now also J7.5 (Pin_5)
- net PD13: now also J7.6 (Pin_6)
- net PD14: now also J7.7 (Pin_7)
- net PD9: now also J7.2 (Pin_2)
- net PE14: now also J7.8 (Pin_8)
- net PE15: now also J7.9 (Pin_9)
- net PF10: now also J10.7 (Pin_7)
- net PF11: now also J10.8 (Pin_8)
- net PF12: now also J10.9 (Pin_9)
- net PF3: now also J7.10 (Pin_10)
- net PF4: now also J10.1 (Pin_1)
- net PF5: now also J10.2 (Pin_2)
- net PF6: now also J10.3 (Pin_3)
- net PF7: now also J10.4 (Pin_4)
- net PF8: now also J10.5 (Pin_5)
- net PF9: now also J10.6 (Pin_6)
- net ESP DEV_KIT J3 pin8: now reaches R32.1
- net ESP DEV_KIT J3 pin8: now also U3.J3-8 (IO19)
- net ESP S3 J3 pin2: now reaches R3.2
- net ESP S3 J3 pin2: now also U4.24 (GPIO43-TX0)
- net ESP DEV_KIT J3 pin19: now reaches R31.1
- net ESP DEV_KIT J3 pin19: now also U3.J3-19 (CLK)
- net ESP DEV_KIT J2 pin17: now reaches R54.2
- net ESP DEV_KIT J2 pin17: now also U3.J2-17 (SD3)
- net ESP DEV_KIT J3 pin9: now reaches R33.1
- net ESP DEV_KIT J3 pin9: now also U3.J3-9 (IO18)
- net ESP DEV_KIT J2 pin12: now reaches R50.2
- net ESP DEV_KIT J2 pin12: now also U3.J2-12 (IO14)
- net ESP S3 J3 pin19: now reaches R20.2
- net ESP S3 J3 pin19: now also U4.41 (GPIO20-D+)
- net ESP DEV_KIT J2 pin2: now reaches R40.2
- net ESP DEV_KIT J2 pin2: now also U3.J2-2 (EN)
- net ESP S3 J1 pin19: now reaches R71.2
- net ESP S3 J1 pin19: now also U4.19 (GPIO13)
- net ESP DEV_KIT J3 pin13: now reaches R37.1
- net ESP DEV_KIT J3 pin13: now also U3.J3-13 (IO4)
- net ESP S3 J3 pin15: now reaches R16.2
- net ESP S3 J3 pin15: now also U4.37 (GPIO45!!!D)
- net ESP S3 J3 pin16: now reaches R17.2
- net ESP S3 J3 pin16: now also U4.38 (GPIO48)
- net ESP S3 J3 pin8: now reaches R9.2
- net ESP S3 J3 pin8: now also U4.30 (GPIO40)
- net ESP S3 J1 pin20: now reaches R72.2
- net ESP S3 J1 pin20: now also U4.20 (GPIO14)
- net ESP DEV_KIT J2 pin15: now reaches R52.2
- net ESP DEV_KIT J2 pin15: now also U3.J2-15 (IO13)
- net ESP DEV_KIT J2 pin13: now reaches R51.2
- net ESP DEV_KIT J2 pin13: now also U3.J2-13 (IO12)
- net ESP S3 J1 pin14: now reaches R66.2
- net ESP S3 J1 pin14: now also U4.14 (GPIO46!!!D)
- net ESP S3 J1 pin18: now reaches R70.2
- net ESP S3 J1 pin18: now also U4.18 (GPIO12)
- net ESP S3 J1 pin10: now reaches R62.2
- net ESP S3 J1 pin10: now also U4.10 (GPIO17-TX1)
- net ESP S3 J1 pin12: now reaches R64.2
- net ESP S3 J1 pin12: now also U4.12 (GPIO8)
- net ESP S3 J1 pin8: now reaches R60.2
- net ESP S3 J1 pin8: now also U4.8 (GPIO15-RTS0)
- net ESP S3 J3 pin10: now reaches R11.2
- net ESP S3 J3 pin10: now also U4.32 (GPIO38)
- net ESP DEV_KIT J3 pin18: now reaches R30.1
- net ESP DEV_KIT J3 pin18: now also U3.J3-18 (SD0)
- net ESP DEV_KIT J2 pin5: now reaches R43.2
- net ESP DEV_KIT J2 pin5: now also U3.J2-5 (IO34)
- net ESP S3 J3 pin4: now reaches R5.2
- net ESP S3 J3 pin4: now also U4.26 (GPIO1)
- net ESP DEV_KIT J3 pin3: now reaches R23.1
- net ESP DEV_KIT J3 pin3: now also U3.J3-3 (IO22)
- net ESP DEV_KIT J3 pin12: now reaches R36.1
- net ESP DEV_KIT J3 pin12: now also U3.J3-12 (IO16)
- net ESP DEV_KIT J2 pin8: now reaches R46.2
- net ESP DEV_KIT J2 pin8: now also U3.J2-8 (IO33)
- net ESP DEV_KIT J3 pin15: now reaches R27.1
- net ESP DEV_KIT J3 pin15: now also U3.J3-15 (IO2)
- net ESP S3 J1 pin5: now reaches R57.2
- net ESP S3 J1 pin5: now also U4.5 (GPIO5)
- net ESP S3 J3 pin9: now reaches R10.2
- net ESP S3 J3 pin9: now also U4.31 (GPIO39)
- net ESP DEV_KIT J3 pin11: now reaches R35.1
- net ESP DEV_KIT J3 pin11: now also U3.J3-11 (IO17)
- net ESP DEV_KIT J2 pin3: now reaches R41.2
- net ESP DEV_KIT J2 pin3: now also U3.J2-3 (SENSOR_VP)
- net ESP DEV_KIT J3 pin10: now reaches R34.1
- net ESP DEV_KIT J3 pin10: now also U3.J3-10 (IO5)
- net ESP S3 J3 pin5: now reaches R6.2
- net ESP S3 J3 pin5: now also U4.27 (GPIO2)
- net ESP S3 J3 pin20: now reaches R21.2
- net ESP S3 J3 pin20: now also U4.42 (GPIO19-D-)
- net ESP S3 J3 pin12: now reaches R13.2
- net ESP S3 J3 pin12: now also U4.34 (GPIO36)
- net ESP S3 J1 pin7: now reaches R59.2
- net ESP S3 J1 pin7: now also U4.7 (GPIO7)
- net at U1.100 (PA8): now also J1.9 (Pin_9)
- net at U1.101 (PA9): now also J1.10 (Pin_10)
- net at C15.1, R2.2, U1.25 (NRST): now also SW1.3 (K), SW1.4 (A)
- net at U1.34 (PA0): now also J1.1 (Pin_1)
- net at U1.35 (PA1): now also J1.2 (Pin_2)
- net at U1.36 (PA2): now also J1.3 (Pin_3)
- net at U1.37 (PA3): now also J1.4 (Pin_4)
- net at U1.40 (PA4): now also J1.5 (Pin_5)
- net at U1.41 (PA5): now also J1.6 (Pin_6)
- net at U1.42 (PA6): now also J1.7 (Pin_7)
- net at U1.43 (PA7): now also J1.8 (Pin_8)
- net ESP S3 J1 pin11: now reaches R63.2
- net ESP S3 J1 pin11: now also U4.11 (GPIO18-RX1)
- net ESP DEV_KIT J2 pin6: now reaches R44.2
- net ESP DEV_KIT J2 pin6: now also U3.J2-6 (IO35)
- net ESP S3 J1 pin9: now reaches R61.2
- net ESP S3 J1 pin9: now also U4.9 (GPIO16-CTS0)
- net ESP DEV_KIT J2 pin16: now reaches R53.2
- net ESP DEV_KIT J2 pin16: now also U3.J2-16 (SD2)
- net ESP DEV_KIT J2 pin10: now reaches R48.2
- net ESP DEV_KIT J2 pin10: now also U3.J2-10 (IO26)
- net ESP DEV_KIT J2 pin9: now reaches R47.2
- net ESP DEV_KIT J2 pin9: now also U3.J2-9 (IO25)
- net ESP S3 J3 pin6: now reaches R7.2
- net ESP S3 J3 pin6: now also U4.28 (GPIO42)
- net ESP S3 J3 pin17: now reaches R18.2
- net ESP S3 J3 pin17: now also U4.39 (GPIO47)
- net ESP DEV_KIT J3 pin5: now reaches R25.1
- net ESP DEV_KIT J3 pin5: now also U3.J3-5 (RXD0)
- net ESP S3 J3 pin7: now reaches R8.2
- net ESP S3 J3 pin7: now also U4.29 (GPIO41)
- net ESP S3 J1 pin4: now reaches R56.2
- net ESP S3 J1 pin4: now also U4.4 (GPIO4)
- net ESP S3 J3 pin11: now reaches R12.2
- net ESP S3 J3 pin11: now also U4.33 (GPIO37)
- net ESP DEV_KIT J2 pin18: now reaches R55.2
- net ESP DEV_KIT J2 pin18: now also U3.J2-18 (CMD)
- net ESP DEV_KIT J3 pin6: now reaches R26.1
- net ESP DEV_KIT J3 pin6: now also U3.J3-6 (IO21)
- net ESP DEV_KIT J2 pin7: now reaches R45.2
- net ESP DEV_KIT J2 pin7: now also U3.J2-7 (IO32)
- net ESP S3 J1 pin6: now reaches R58.2
- net ESP S3 J1 pin6: now also U4.6 (GPIO6)
- net ESP S3 J1 pin13: now reaches R65.2
- net ESP S3 J1 pin13: now also U4.13 (GPIO3!!!D)
- net ESP S3 J1 pin17: now reaches R69.2
- net ESP S3 J1 pin17: now also U4.17 (GPIO11)
- net ESP S3 J3 pin3: now reaches R4.2
- net ESP S3 J3 pin3: now also U4.25 (GPIO44-RX0)
- net ESP DEV_KIT J3 pin14: now reaches R38.1
- net ESP DEV_KIT J3 pin14: now also U3.J3-14 (IO0)
- net ESP DEV_KIT J3 pin4: now reaches R24.1
- net ESP DEV_KIT J3 pin4: now also U3.J3-4 (TXD0)
- net ESP DEV_KIT J3 pin17: now reaches R29.1
- net ESP DEV_KIT J3 pin17: now also U3.J3-17 (SD1)
- net ESP S3 J1 pin15: now reaches R67.2
- net ESP S3 J1 pin15: now also U4.15 (GPIO9)
- net ESP S3 J1 pin16: now reaches R68.2
- net ESP S3 J1 pin16: now also U4.16 (GPIO10)
- net ESP S3 J3 pin14: now reaches R15.2
- net ESP S3 J3 pin14: now also U4.36 (GPIO0!!!U)
- net ESP S3 J3 pin18: now reaches R19.2
- net ESP S3 J3 pin18: now also U4.40 (GPIO21)
- net ESP DEV_KIT J2 pin4: now reaches R42.2
- net ESP DEV_KIT J2 pin4: now also U3.J2-4 (SENSOR_VN)
- net ESP DEV_KIT J3 pin2: now reaches R22.1
- net ESP DEV_KIT J3 pin2: now also U3.J3-2 (IO23)
- net ESP DEV_KIT J3 pin16: now reaches R28.1
- net ESP DEV_KIT J3 pin16: now also U3.J3-16 (IO15)
- net ESP S3 J3 pin13: now reaches R14.2
- net ESP S3 J3 pin13: now also U4.35 (GPIO35)
- net ESP DEV_KIT J2 pin11: now reaches R49.2
- net ESP DEV_KIT J2 pin11: now also U3.J2-11 (IO27)
- new net: U4.1 (3V3), U4.2 (3V3)
- no-connect marks 16 -> 20
Other:
- removed sheet Sheet: shield for esp32 S3 and esp32 dev kit
- note added: "ESP32-DEVKITC"
- note added: "ESP32-S3"
