File: Univerzalni_testovaci_platforma_nejen_pro_IoT_v1/Univerzalni_testovaci_platforma_nejen_pro_IoT_v1.kicad_pcb (KiCad board)
At the start: 4 copper layers, 100 x 100 mm, 113 parts, among them J1 Conn_01x22_Female ESP S3, J2 Conn_01x22_Female ESP S3, J3 Conn_01x19_Female ESP DEV_KIT, J4 Conn_01x19_Female ESP DEV_KIT, J5 Conn_02x03_Counter_Clockwise, J6 USB_C_Receptacle, J7 Conn_02x10_Odd_Even, J8 Conn_02x10_Odd_Even, SW1 SW_Push_Dual, U1 STM32F103ZETx, U2 AMS1117CS-3.3, Y1 12Mhz

Commit message: schema hotovo
Parts:
- added H1: MountingHole, MountingHole:MountingHole_3.2mm_M3, F.Cu at (103.9, 54.2)
- added H2: MountingHole, MountingHole:MountingHole_3.2mm_M3, F.Cu at (196.3, 53.7)
- added H3: MountingHole, MountingHole:MountingHole_3.2mm_M3, F.Cu at (196.2, 146.2)
- added H4: MountingHole, MountingHole:MountingHole_3.2mm_M3, F.Cu at (103.7, 146.3)
- added J10: Conn_01x10_Male, Connector_PinHeader_2.54mm:PinHeader_1x10_P2.54mm_Vertical, F.Cu at (143.8, 157.2)
- added J11: Conn_01x10_Male, Connector_PinHeader_2.54mm:PinHeader_1x10_P2.54mm_Vertical, F.Cu at (71.3, 156.5)
- added J12: Conn_01x10_Male, Connector_PinHeader_2.54mm:PinHeader_1x10_P2.54mm_Vertical, F.Cu at (126.0, 157.3)
- added J9: Conn_01x10_Male, Connector_PinHeader_2.54mm:PinHeader_1x10_P2.54mm_Vertical, F.Cu at (153.9, 157.2)
- added U3: ESP32-DEVKITC-32D, robotarna:MODULE_ESP32-DEVKITC-32D, F.Cu at (114.5, 80.6)
- added U4: ESP32-S3, robotarna1:ESP32-devkit_v1, F.Cu at (186.9, 59.0)
- J1, J2: value Conn_01x22_Female ESP S3 -> Conn_01x10_Male; footprint Connector_PinSocket_2.54mm:PinSocket_1x22_P2.54mm_Vertical -> Connector_PinHeader_2.54mm:PinHeader_1x10_P2.54mm_Vertical
- J3, J4: value Conn_01x19_Female ESP DEV_KIT -> Conn_01x10_Male; footprint Connector_PinSocket_2.54mm:PinSocket_1x19_P2.54mm_Vertical -> Connector_PinHeader_2.54mm:PinHeader_1x10_P2.54mm_Vertical
- J7, J8: value Conn_02x10_Odd_Even -> Conn_01x10_Male; footprint Connector_PinHeader_2.54mm:PinHeader_2x10_P2.54mm_Vertical -> Connector_PinHeader_2.54mm:PinHeader_1x10_P2.54mm_Vertical
- U2: value AMS1117CS-3.3 -> AMS1117-3.3
- moved D2 130.4 mm to (147.9, 140.1), turned to -90 degrees
- moved U2 127.8 mm to (136.8, 141.0), turned to 0 degrees
- moved J3 116.8 mm to (147.2, 157.2)
- moved J2 112.0 mm to (140.5, 157.2)
- moved J4 110.8 mm to (137.2, 157.2)
- moved C18 108.7 mm to (136.5, 132.3), turned to 180 degrees
- moved R3 108.1 mm to (148.6, 127.5)
- moved R74 105.8 mm to (132.0, 136.7)
- moved J1 105.3 mm to (130.0, 157.2)
- moved C17 104.2 mm to (129.0, 140.9), turned to 90 degrees
- moved J8 97.9 mm to (76.0, 156.6), turned to 0 degrees
- moved J7 43.6 mm to (133.8, 157.2), turned to 0 degrees
- moved SW1 20.9 mm to (104.9, 137.5)
- moved J6 8.20 mm to (120.6, 145.8)
- moved R75 8.20 mm to (119.3, 137.0)
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Connections:
- J1 pad 1: Net-(J1-Pad1) -> Net-(U1-Pad34)
- J1 pad 10: Net-(J1-Pad10) -> Net-(U1-Pad101)
- J1 pad 2: Net-(J1-Pad1) -> Net-(U1-Pad35)
- J1 pad 3: unconnected-(J1-Pad3) -> Net-(U1-Pad36)
- J1 pad 4: Net-(J1-Pad4) -> Net-(U1-Pad37)
- J1 pad 5: Net-(J1-Pad5) -> Net-(U1-Pad40)
- J1 pad 6: Net-(J1-Pad6) -> Net-(U1-Pad41)
- J1 pad 7: Net-(J1-Pad7) -> Net-(U1-Pad42)
- J1 pad 8: Net-(J1-Pad8) -> Net-(U1-Pad43)
- J1 pad 9: Net-(J1-Pad9) -> Net-(U1-Pad100)
- J2 pad 1: GND -> PA10
- J2 pad 10: Net-(J2-Pad10) -> PC7
- J2 pad 2: Net-(J2-Pad2) -> PA13
- J2 pad 3: Net-(J2-Pad3) -> PA14
- J2 pad 4: Net-(J2-Pad4) -> PA15
- J2 pad 5: Net-(J2-Pad5) -> PB0
- J2 pad 6: Net-(J2-Pad6) -> PB1
- J2 pad 7: Net-(J2-Pad7) -> PC4
- J2 pad 8: Net-(J2-Pad8) -> PC5
- J2 pad 9: Net-(J2-Pad9) -> PC6
- J3 pad 1: +3V3 -> GND
- J3 pad 10: Net-(J3-Pad10) -> GND
- J3 pad 2: Net-(J3-Pad2) -> GND
- J3 pad 3: Net-(J3-Pad3) -> GND
- J3 pad 4: Net-(J3-Pad4) -> GND
- J3 pad 5: Net-(J3-Pad5) -> GND
- J3 pad 6: Net-(J3-Pad6) -> GND
- J3 pad 7: Net-(J3-Pad7) -> GND
- J3 pad 8: Net-(J3-Pad8) -> GND
- J3 pad 9: Net-(J3-Pad9) -> GND
- J4 pad 10: Net-(J4-Pad10) -> GND
- J4 pad 2: Net-(J4-Pad2) -> GND
- J4 pad 3: Net-(J4-Pad3) -> GND
- J4 pad 4: Net-(J4-Pad4) -> GND
- J4 pad 5: Net-(J4-Pad5) -> GND
- J4 pad 6: Net-(J4-Pad6) -> GND
- J4 pad 8: Net-(J4-Pad8) -> GND
- J4 pad 9: Net-(J4-Pad9) -> GND
- J7 pad 1: Net-(U1-Pad34) -> PC8
- J7 pad 10: PB0 -> PF3
- J7 pad 2: PA10 -> PD9
- J7 pad 3: Net-(U1-Pad35) -> PD10
- J7 pad 4: PA13 -> PD11
- J7 pad 5: Net-(U1-Pad36) -> PD12
- J7 pad 6: PA14 -> PD13
- J7 pad 7: Net-(U1-Pad37) -> PD14
- J7 pad 8: PA15 -> PE14
- J7 pad 9: Net-(U1-Pad40) -> PE15
- J8 pad 1: PC8 -> GND
- J8 pad 10: PF8 -> GND
- J8 pad 2: PF4 -> GND
- J8 pad 3: PD9 -> GND
- J8 pad 4: PF5 -> GND
- J8 pad 5: PD10 -> GND
- J8 pad 6: PF6 -> GND
- J8 pad 7: PD11 -> GND
- J8 pad 8: PF7 -> GND
- J8 pad 9: PD12 -> GND
- R10 pad 2: Net-(J2-Pad9) -> /ESP S3 J3 pin9
- R11 pad 2: Net-(J2-Pad10) -> /ESP S3 J3 pin10
- R12 pad 2: Net-(J2-Pad11) -> /ESP S3 J3 pin11
- R13 pad 2: Net-(J2-Pad12) -> /ESP S3 J3 pin12
- R14 pad 2: Net-(J2-Pad13) -> /ESP S3 J3 pin13
- R15 pad 2: Net-(J2-Pad14) -> /ESP S3 J3 pin14
- R16 pad 2: Net-(J2-Pad15) -> /ESP S3 J3 pin15
- R17 pad 2: Net-(J2-Pad16) -> /ESP S3 J3 pin16
- R18 pad 2: Net-(J2-Pad17) -> /ESP S3 J3 pin17
- R19 pad 2: Net-(J2-Pad18) -> /ESP S3 J3 pin18
- R20 pad 2: Net-(J2-Pad19) -> /ESP S3 J3 pin19
- R21 pad 2: Net-(J2-Pad20) -> /ESP S3 J3 pin20
- R22 pad 1: Net-(J4-Pad2) -> /ESP DEV_KIT J3 pin2
- R23 pad 1: Net-(J4-Pad3) -> /ESP DEV_KIT J3 pin3
- R24 pad 1: Net-(J4-Pad4) -> /ESP DEV_KIT J3 pin4
- R25 pad 1: Net-(J4-Pad5) -> /ESP DEV_KIT J3 pin5
- R26 pad 1: Net-(J4-Pad6) -> /ESP DEV_KIT J3 pin6
- R27 pad 1: Net-(J4-Pad15) -> /ESP DEV_KIT J3 pin15
- R28 pad 1: Net-(J4-Pad16) -> /ESP DEV_KIT J3 pin16
- R29 pad 1: Net-(J4-Pad17) -> /ESP DEV_KIT J3 pin17
- R3 pad 2: Net-(J2-Pad2) -> /ESP S3 J3 pin2
- R30 pad 1: Net-(J4-Pad18) -> /ESP DEV_KIT J3 pin18
- R31 pad 1: Net-(J4-Pad19) -> /ESP DEV_KIT J3 pin19
- R32 pad 1: Net-(J4-Pad8) -> /ESP DEV_KIT J3 pin8
- R33 pad 1: Net-(J4-Pad9) -> /ESP DEV_KIT J3 pin9
- R34 pad 1: Net-(J4-Pad10) -> /ESP DEV_KIT J3 pin10
- R35 pad 1: Net-(J4-Pad11) -> /ESP DEV_KIT J3 pin11
- R36 pad 1: Net-(J4-Pad12) -> /ESP DEV_KIT J3 pin12
- R37 pad 1: Net-(J4-Pad13) -> /ESP DEV_KIT J3 pin13
- R38 pad 1: Net-(J4-Pad14) -> /ESP DEV_KIT J3 pin14
- R4 pad 2: Net-(J2-Pad3) -> /ESP S3 J3 pin3
- R40 pad 2: Net-(J3-Pad2) -> /ESP DEV_KIT J2 pin2
- R41 pad 2: Net-(J3-Pad3) -> /ESP DEV_KIT J2 pin3
- R42 pad 2: Net-(J3-Pad4) -> /ESP DEV_KIT J2 pin4
- R43 pad 2: Net-(J3-Pad5) -> /ESP DEV_KIT J2 pin5
- R44 pad 2: Net-(J3-Pad6) -> /ESP DEV_KIT J2 pin6
- R45 pad 2: Net-(J3-Pad7) -> /ESP DEV_KIT J2 pin7
- R46 pad 2: Net-(J3-Pad8) -> /ESP DEV_KIT J2 pin8
- R47 pad 2: Net-(J3-Pad9) -> /ESP DEV_KIT J2 pin9
- R48 pad 2: Net-(J3-Pad10) -> /ESP DEV_KIT J2 pin10
- R49 pad 2: Net-(J3-Pad11) -> /ESP DEV_KIT J2 pin11
- R5 pad 2: Net-(J2-Pad4) -> /ESP S3 J3 pin4
- R50 pad 2: Net-(J3-Pad12) -> /ESP DEV_KIT J2 pin12
- R51 pad 2: Net-(J3-Pad13) -> /ESP DEV_KIT J2 pin13
- R52 pad 2: Net-(J3-Pad15) -> /ESP DEV_KIT J2 pin15
- R53 pad 2: Net-(J3-Pad16) -> /ESP DEV_KIT J2 pin16
- R54 pad 2: Net-(J3-Pad17) -> /ESP DEV_KIT J2 pin17
- R55 pad 2: Net-(J3-Pad18) -> /ESP DEV_KIT J2 pin18
- R56 pad 2: Net-(J1-Pad4) -> /ESP S3 J1 pin4
- R57 pad 2: Net-(J1-Pad5) -> /ESP S3 J1 pin5
- R58 pad 2: Net-(J1-Pad6) -> /ESP S3 J1 pin6
- R59 pad 2: Net-(J1-Pad7) -> /ESP S3 J1 pin7
- R6 pad 2: Net-(J2-Pad5) -> /ESP S3 J3 pin5
- R60 pad 2: Net-(J1-Pad8) -> /ESP S3 J1 pin8
- R61 pad 2: Net-(J1-Pad9) -> /ESP S3 J1 pin9
- R62 pad 2: Net-(J1-Pad10) -> /ESP S3 J1 pin10
- R63 pad 2: Net-(J1-Pad11) -> /ESP S3 J1 pin11
- R64 pad 2: Net-(J1-Pad12) -> /ESP S3 J1 pin12
- R65 pad 2: Net-(J1-Pad13) -> /ESP S3 J1 pin13
- R66 pad 2: Net-(J1-Pad14) -> /ESP S3 J1 pin14
- R67 pad 2: Net-(J1-Pad15) -> /ESP S3 J1 pin15
- R68 pad 2: Net-(J1-Pad16) -> /ESP S3 J1 pin16
- R69 pad 2: Net-(J1-Pad17) -> /ESP S3 J1 pin17
- R7 pad 2: Net-(J2-Pad6) -> /ESP S3 J3 pin6
- R70 pad 2: Net-(J1-Pad18) -> /ESP S3 J1 pin18
- R71 pad 2: Net-(J1-Pad19) -> /ESP S3 J1 pin19
- R72 pad 2: Net-(J1-Pad20) -> /ESP S3 J1 pin20
- R79 pad 1: +5V -> +3V3
- R8 pad 2: Net-(J2-Pad7) -> /ESP S3 J3 pin7
- R9 pad 2: Net-(J2-Pad8) -> /ESP S3 J3 pin8
- U2 pad 3: +3V3 -> +5V
Routing:
- net +5V: track 0.00 -> 15.1 mm
- net GND: track 9.66 -> 11.3 mm, vias 0 -> 3
- added copper zone on In1.Cu, net +3V3
- added copper zone on In2.Cu, net GND

Commit message: asi hotovo
Parts:
- removed JP1: Jumper_2_Open, Connector_PinHeader_2.54mm:PinHeader_1x02_P2.54mm_Vertical
- moved R17 160.1 mm to (195.2, 97.1)
- moved R16 160.0 mm to (195.1, 94.6)
- moved R7 156.6 mm to (195.1, 71.7)
- moved R9 154.5 mm to (195.1, 76.8)
- moved R12 151.6 mm to (195.1, 84.4)
- moved R11 149.9 mm to (195.1, 81.9)
- moved R5 145.3 mm to (195.1, 66.6)
- moved R18 144.2 mm to (195.2, 99.6)
- moved R64 142.6 mm to (178.7, 86.9), turned to 180 degrees
- moved R21 141.7 mm to (195.1, 107.2)
- moved D1 140.9 mm to (151.9, 147.4), turned to 180 degrees
- moved R13 140.1 mm to (195.1, 86.9)
- moved R20 139.3 mm to (195.0, 104.7)
- moved R19 137.1 mm to (195.2, 102.2)
- moved R70 133.1 mm to (178.6, 102.2), turned to 180 degrees
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Routing:
- net Net-(R70-Pad1): track 0.00 -> 139.1 mm, vias 0 -> 4
- net Net-(R71-Pad1): track 0.00 -> 138.5 mm, vias 0 -> 4
- net Net-(R72-Pad1): track 0.00 -> 137.9 mm, vias 0 -> 4
- net Net-(R69-Pad1): track 0.00 -> 137.4 mm, vias 0 -> 4
- net Net-(R40-Pad1): track 0.00 -> 132.0 mm
- net Net-(R19-Pad1): track 0.00 -> 130.8 mm, vias 0 -> 2
- net Net-(R20-Pad1): track 0.00 -> 130.7 mm, vias 0 -> 2
- net Net-(R21-Pad1): track 0.00 -> 128.6 mm, vias 0 -> 2
- net Net-(R17-Pad1): track 0.00 -> 126.4 mm, vias 0 -> 2
- net Net-(R16-Pad1): track 0.00 -> 122.9 mm, vias 0 -> 2
- net Net-(C15-Pad1): track 0.00 -> 118.7 mm, vias 0 -> 3
- net Net-(R5-Pad1): track 0.00 -> 118.1 mm, vias 0 -> 2
- net Net-(R14-Pad1): track 0.00 -> 118.1 mm, vias 0 -> 2
- net Net-(R15-Pad1): track 0.00 -> 117.6 mm, vias 0 -> 2
- net Net-(R12-Pad1): track 0.00 -> 117.3 mm, vias 0 -> 2
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
Commit message: uplně hotovo
Parts:
- moved J11 3.80 mm to (106.2, 111.5)
- moved J3 3.70 mm to (102.5, 111.5)
- moved J12 3.70 mm to (196.8, 129.0)
- moved J4 3.70 mm to (196.8, 132.7)
Routing:
- net unconnected-(J6-PadS1): track 0.00 -> 17.0 mm
- net +5V: track 15.1 -> 20.2 mm, vias 0 -> 2
- net Net-(J6-PadA7): track 8.64 -> 11.9 mm
- net Net-(J6-PadA6): track 8.85 -> 12.1 mm
- net unconnected-(U4-Pad1): track 0.00 -> 2.54 mm
- net GND: track 114.6 -> 117.1 mm, vias 29 -> 30
- net /ESP DEV_KIT J2 pin12: track 0.00 -> 2.40 mm
- net /ESP DEV_KIT J3 pin8: track 0.00 -> 2.30 mm
- net Net-(C15-Pad1): track 118.7 -> 116.4 mm, vias 3 -> 2
- net /ESP DEV_KIT J3 pin9: track 0.00 -> 2.20 mm
- net Net-(R14-Pad1): track 118.1 -> 117.2 mm
- added copper zone on B.Cu, net GND
- added copper zone on F.Cu, net GND

Commit message: jdu to objednat
Parts:
- added J13: Conn_01x10_Male, Connector_PinHeader_2.54mm:PinHeader_1x10_P2.54mm_Vertical, F.Cu at (155.1, 65.9)
- D1: value BLUE -> RED
- moved J3 2.40 mm to (104.9, 111.5)
- moved J4 2.40 mm to (196.8, 130.3)
- moved J11 1.20 mm to (107.4, 111.5)
- moved J12 1.20 mm to (196.8, 127.8)
- moved J9 1.20 mm to (155.1, 68.4)
Routing:
- net +3V3: track 72.1 -> 194.5 mm, vias 15 -> 81
- net GND: track 117.1 -> 97.4 mm, vias 30 -> 24
- net +3.3VA: track 3.64 -> 7.49 mm, vias 0 -> 3

Commit message: změny schématu pro lepší focení
Changed lines of the file:
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@@
       (sketchpadsonfab false)
       (subtractmaskfromsilk false)
-      (outputformat 1)
+      (outputformat 4)
       (mirror false)
-      (drillshape 1)
+      (drillshape 0)
       (scaleselection 1)
       (outputdirectory "")
@@
     (fp_line (start -1 -0.625) (end 1 -0.625) (layer "F.Fab") (width 0.1))
     (fp_line (start 1 -0.625) (end 1 0.625) (layer "F.Fab") (width 0.1))
-    (pad "1" smd roundrect (at -1.0375 0 270) (size 1.175 1.45) (layers "F.Cu" "F.Paste" "F.Mask") (roundrect_rratio 0.212766)
+    (pad "1" smd roundrect (at -1.0375 0 270) (size 1.175 1.45) (layers "F.Cu" "F.Paste" "F.Mask") (roundrect_rratio 0.2127659574)
       (net 1 "+3V3") (pintype "passive"))
-    (pad "2" smd roundrect (at 1.0375 0 270) (size 1.175 1.45) (layers "F.Cu" "F.Paste" "F.Mask") (roundrect_rratio 0.212766)
+    (pad "2" smd roundrect (at 1.0375 0 270) (size 1.175 1.45) (layers "F.Cu" "F.Paste" "F.Mask") (roundrect_rratio 0.2127659574)
       (net 2 "GND") (pintype "passive"))
     (model "${KICAD6_3DMODEL_DIR}/Capacitor_SMD.3dshapes/C_0805_2012Metric.wrl"
@@
     (fp_line (start -1 0.625) (end -1 -0.625) (layer "F.Fab") (width 0.1))
     (fp_line (start -1 -0.625) (end 1 -0.625) (layer "F.Fab") (width 0.1))
-    (pad "1" smd roundrect (at -1.0375 0 270) (size 1.175 1.45) (layers "F.Cu" "F.Paste" "F.Mask") (roundrect_rratio 0.212766)
+    (pad "1" smd roundrect (at -1.0375 0 270) (size 1.175 1.45) (layers "F.Cu" "F.Paste" "F.Mask") (roundrect_rratio 0.2127659574)
       (net 1 "+3V3") (pintype "passive"))
-    (pad "2" smd roundrect (at 1.0375 0 270) (size 1.175 1.45) (layers "F.Cu" "F.Paste" "F.Mask") (roundrect_rratio 0.212766)
+    (pad "2" smd roundrect (at 1.0375 0 270) (size 1.175 1.45) (layers "F.Cu" "F.Paste" "F.Mask") (roundrect_rratio 0.2127659574)
       (net 2 "GND") (pintype "passive"))
     (model "${KICAD6_3DMODEL_DIR}/Capacitor_SMD.3dshapes/C_0805_2012Metric.wrl"
@@
     (fp_line (start 1 -0.625) (end 1 0.625) (layer "F.Fab") (width 0.1))
     (fp_line (start 1 0.625) (end -1 0.625) (layer "F.Fab") (width 0.1))
-    (pad "1" smd roundrect (at -1.0375 0 90) (size 1.175 1.45) (layers "F.Cu" "F.Paste" "F.Mask") (roundrect_rratio 0.212766)
+    (pad "1" smd roundrect (at -1.0375 0 90) (size 1.175 1.45) (layers "F.Cu" "F.Paste" "F.Mask") (roundrect_rratio 0.2127659574)
       (net 3 "+3.3VA") (pintype "passive"))
-    (pad "2" smd roundrect (at 1.0375 0 90) (size 1.175 1.45) (layers "F.Cu" "F.Paste" "F.Mask") (roundrect_rratio 0.212766)
+    (pad "2" smd roundrect (at 1.0375 0 90) (size 1.175 1.45) (layers "F.Cu" "F.Paste" "F.Mask") (roundrect_rratio 0.2127659574)
       (net 2 "GND") (pintype "passive"))
     (model "${KICAD6_3DMODEL_DIR}/Capacitor_SMD.3dshapes/C_0805_2012Metric.wrl"
@@
     (fp_line (start 1 -0.625) (end 1 0.625) (layer "F.Fab") (width 0.1))
     (fp_line (start -1 -0.625) (end 1 -0.625) (layer "F.Fab") (width 0.1))
-    (pad "1" smd roundrect (at -1.0375 0 90) (size 1.175 1.45) (layers "F.Cu" "F.Paste" "F.Mask") (roundrect_rratio 0.212766)
+    (pad "1" smd roundrect (at -1.0375 0 90) (size 1.175 1.45) (layers "F.Cu" "F.Paste" "F.Mask") (roundrect_rratio 0.2127659574)
       (net 1 "+3V3") (pintype "passive"))
-    (pad "2" smd roundrect (at 1.0375 0 90) (size 1.175 1.45) (layers "F.Cu" "F.Paste" "F.Mask") (roundrect_rratio 0.212766)
+    (pad "2" smd roundrect (at 1.0375 0 90) (size 1.175 1.45) (layers "F.Cu" "F.Paste" "F.Mask") (roundrect_rratio 0.2127659574)
       (net 2 "GND") (pintype "passive"))
     (model "${KICAD6_3DMODEL_DIR}/Capacitor_SMD.3dshapes/C_0805_2012Metric.wrl"
@@
     (fp_line (start -2.2 -1.6) (end -3 -0.8) (layer "F.Fab") (width 0.1))
     (fp_line (start 3 -1.6) (end -2.2 -1.6) (layer "F.Fab") (width 0.1))
-    (pad "1" smd roundrect (at -2.55 0 270) (size 2.25 2.35) (layers "F.Cu" "F.Paste" "F.Mask") (roundrect_rratio 0.111111)
+    (pad "1" smd roundrect (at -2.55 0 270) (size 2.25 2.35) (layers "F.Cu" "F.Paste" "F.Mask") (roundrect_rratio 0.1111111111)
       (net 1 "+3V3") (pintype "passive"))
-    (pad "2" smd roundrect (at 2.55 0 270) (size 2.25 2.35) (layers "F.Cu" "F.Paste" "F.Mask") (roundrect_rratio 0.111111)
+    (pad "2" smd roundrect (at 2.55 0 270) (size 2.25 2.35) (layers "F.Cu" "F.Paste" "F.Mask") (roundrect_rratio 0.1111111111)
       (net 2 "GND") (pintype "passive"))
     (model "${KICAD6_3DMODEL_DIR}/Capacitor_Tantalum_SMD.3dshapes/CP_EIA-6032-20_AVX-F.wrl"
